File: Estado_GPIO.kicad_sch (KiCad schematic)
At the start: 56 parts

Commit message: Actualización Modulo RPI
Parts:
- added D31 (x2): LED, LED_SMD:LED_1206_3216Metric, symbol Device:LED
- added R31: 10K, Resistor_SMD:R_1206_3216Metric, symbol Device:R
- added R31: 1K, Resistor_SMD:R_1206_3216Metric, symbol Device:R
- D30, D32: Enlace de compra (none) -> https://www.vistronica.com/componentes-activos/diodos/led/l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; Package (none) -> 1206
- R2, R32: Enlace de compra (none) -> https://www.vistronica.com/componentes-pasivos/resistencias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; Package (none) -> 1206
Connections:
- net GND: now also D31.1 (K), D31.1 (K)
- new net: D31.2 (A), R31.2 (x2)
- new net 5V: R31.1
- new net RTC: R31.1
Other:
- moved on the sheet: D30, D32, R2, R32
