File: Module_RPI.kicad_pcb (KiCad board)
At the start: 2 copper layers, 110.2 x 79.8 mm, 159 parts, among them J1_Rele1 Conn_02x20_Odd_Even, J2 Conn_01x20, J4 Conn_01x20, U2 RASPBERRY_PI_4B_4GB

Commit message: Actualización Modulo RPI
Parts:
- added BT1: Battery, Battery:BatteryHolder_Seiko_MS621F, B.Cu at (63.1, 64.0)
- added C1: 100nF, Capacitor_SMD:C_0805_2012Metric, B.Cu at (63.1, 61.7)
- added C2: 100nF, Capacitor_SMD:C_0805_2012Metric, F.Cu at (91.7, 79.3)
- added J1: Conn_01x02_Pin, Connector_PinHeader_2.54mm:PinHeader_1x02_P2.54mm_Vertical, F.Cu at (53.7, 81.7)
- added R1: 4.7K, Resistor_SMD:R_1206_3216Metric, F.Cu at (89.0, 84.5)
- added R59: 4.7K, Resistor_SMD:R_1206_3216Metric, F.Cu at (92.5, 84.5)
- added R60: 10K, Resistor_SMD:R_1206_3216Metric, F.Cu at (57.8, 81.6)
- added R61: 10K, Resistor_SMD:R_1206_3216Metric, F.Cu at (57.8, 84.2)
- added R62: 10K, Resistor_SMD:R_1206_3216Metric, F.Cu at (89.4, 67.1)
- added RESET RTC: SW_Push, Button_Switch_SMD:SW_SPST_TL3342, F.Cu at (80.0, 62.0)
- added RTC: LED, LED_SMD:LED_1206_3216Metric, F.Cu at (89.5, 69.7)
- added RTC: Jumper_2_Open, Jumper:SolderJumper-2_P1.3mm_Open_RoundedPad1.0x1.5mm, F.Cu at (84.8, 80.3)
- added U1: DS3231M, Package_SO:SOIC-16W_7.5x10.3mm_P1.27mm, F.Cu at (74.0, 72.3)
Routing:
- net GND: track 717.9 -> 804.2 mm, vias 37 -> 39
- net RTC: track 0.00 -> 76.8 mm, vias 0 -> 7
- net BAT: track 0.00 -> 43.9 mm, vias 0 -> 1
- net 32KHz: track 0.00 -> 42.1 mm, vias 0 -> 2
- net GPIO_5: track 40.0 -> 79.8 mm, vias 0 -> 3
- net SQW: track 0.00 -> 32.3 mm, vias 0 -> 2
- net GPIO_3: track 45.1 -> 67.7 mm, vias 0 -> 2
- net Net-(U1-~{RST}): track 0.00 -> 11.0 mm
- net 3.3V: track 224.4 -> 228.0 mm
- net Net-(D1-A): track 0.00 -> 2.64 mm
Other:
- board text added: "32KHz"
- board text added: "Diseñado por Daniel.Gómez para CI24 - 2024"
- board text added: "Modulo RPi"
- board text added: "Protector Extensor GPIO"
- board text added: "Rev 1.0"
- board text added: "SQW"
- board text added: "© Controles inteligentes - 2024."
- board text removed: "Modulo Raspberry"
- board text removed: "© CI24 2024."
