File: Module_RPI.kicad_sch (KiCad schematic)
At the start: 17 parts, among them J1_Rele1 Conn_02x20_Odd_Even, J2 Conn_01x20, J4 Conn_01x20, U2 RASPBERRY_PI_4B_4GB

Commit message: Actualización Modulo RPI
Parts:
- removed D31: LED, LED_SMD:LED_1206_3216Metric, symbol Device:LED
- removed R31: 1K, Resistor_SMD:R_1206_3216Metric, symbol Device:R
- added BT1: Battery, Battery:BatteryHolder_Seiko_MS621F, symbol Device:Battery
- added C1, C2: 100nF, Capacitor_SMD:C_0805_2012Metric, symbol Device:C
- added J1: Conn_01x02_Pin, Connector_PinHeader_2.54mm:PinHeader_1x02_P2.54mm_Vertical, symbol Connector:Conn_01x02_Pin
- added JP30: Jumper_2_Open, Jumper:SolderJumper-2_P1.3mm_Open_RoundedPad1.0x1.5mm, symbol Jumper:Jumper_2_Open
- added R1, R59: 4.7K, Resistor_SMD:R_1206_3216Metric, symbol Device:R
- added R60, R61: 10K, Resistor_SMD:R_1206_3216Metric, symbol Device:R
- added SW1: SW_Push, Button_Switch_SMD:SW_SPST_TL3342, symbol Switch:SW_Push
- added U1: DS3231M, Package_SO:SOIC-16W_7.5x10.3mm_P1.27mm, symbol Timer_RTC:DS3231M
- 3.3V1, 3.3V2, 5V1, 5V2: Package (none) -> THT 2.54mm
- GPIO16, GPIO18, GPIO22, GPIO24, GPIO26, GPIO28, GPIO29: Package (none) -> THT
- J1_Rele1, J2, J4: Enlace de compra (none) -> https://www.vistronica.com/conectores-cables-y-switches/reg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; Package (none) -> THT
- U2: Enlace de compra (none) -> https://www.vistronica.com/conectores-cables-y-switches/reg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
Connections:
- net +3.3V: now also JP30.2 (B)
- net GND: now also BT1.2 (-), C1.2, C2.2, SW1.2, U1.10 (GND), U1.11 (GND), U1.12 (GND), U1.13 (GND), U1.5 (GND), U1.6 (GND), U1.7 (GND), U1.8 (GND), U1.9 (GND)
- net GPIO_3: now also R1.2, U1.16 (SCL)
- net GPIO_5: now also R59.2, U1.15 (SDA)
- new net: SW1.1, U1.4 (~{RST})
- new net 32KHz: J1.2 (Pin_2), R61.2, U1.1 (32KHZ)
- new net BAT: BT1.1 (+), C1.1, U1.14 (VBAT)
- new net RTC: C2.1, JP30.1 (A), R1.1, R59.1, R60.1, R61.1, U1.2 (VCC)
- new net SQW: J1.1 (Pin_1), R60.2, U1.3 (~{INT}/SQW)
- no-connect marks 0 -> 4
Other:
- note added: "ALIMENTACIÓN"
- note added: "RTC"
- note removed: "ALIMENTACION"
- moved on the sheet: 3.3V1, 3.3V2, 5V1, 5V2
