File: Protección_RPO_GPIO.kicad_sch (KiCad schematic)
At the start: 84 parts

Commit message: Actualización Modulo RPI
Parts:
- D3: Enlace de compra (none) -> https://www.vistronica.com/nuevo-compras-diodo-zener-33v-bz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; Package (none) -> SOD-123F
- JP1, JP10, JP11, JP12, JP13, JP14, JP15, JP16, JP17, JP18, JP19, JP2, JP20, JP21, JP22, JP23, JP24, JP25, JP26, JP27, JP28, JP3, JP4, JP5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: Package (none) -> None
- R3: Enlace de compra (none) -> https://www.vistronica.com/componentes-pasivos/resistencias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; Package (none) -> 1206
